File: multiprotocol_nano/multiprotocol_nano.sch (KiCad schematic (older format))
At the start: 7 parts, among them J1 Conn_01x05, J3 Conn_01x03, U1 NRF24L01_Breakout

Commit message: Fix wrong package for LM317
Parts:
- added R2: 1.2K, Resistor_SMD:R_0805_2012Metric_Pad1.15x1.40mm_HandSolder, symbol Device:R
- added R3: 240, Resistor_SMD:R_0805_2012Metric_Pad1.15x1.40mm_HandSolder, symbol Device:R
- added U2: LM317_3PinPackage, Package_TO_SOT_THT:TO-220-3_Vertical, symbol Regulator_Linear:LM317_3PinPackage
- R1, R5: footprint Resistor_THT:R_Axial_DIN0207_L6.3mm_D2.5mm_P10.16mm_Horizontal -> Resistor_SMD:R_0805_2012Metric_Pad1.15x1.40mm_HandSolder
Connections:
- net labels added: VCC
- wire segments 30 -> 40
- no-connect marks 3 -> 23
Changed lines of the file:
@@
 F 0 "R5" V 2643 4850 50  0000 C CNN
 F 1 "10K" V 2734 4850 50  0000 C CNN
-F 2 "Resistor_THT:R_Axial_DIN0207_L6.3mm_D2.5mm_P10.16mm_Horizontal" V 2780 4850 50  0001 C CNN
+F 2 "Resistor_SMD:R_0805_2012Metric_Pad1.15x1.40mm_HandSolder" V 2780 4850 50  0001 C CNN
 F 3 "~" H 2850 4850 50  0001 C CNN
 	1    2850 4850
@@
 F 0 "R1" V 2343 5200 50  0000 C CNN
 F 1 "10K" V 2434 5200 50  0000 C CNN
-F 2 "Resistor_THT:R_Axial_DIN0207_L6.3mm_D2.5mm_P10.16mm_Horizontal" V 2480 5200 50  0001 C CNN
+F 2 "Resistor_SMD:R_0805_2012Metric_Pad1.15x1.40mm_HandSolder" V 2480 5200 50  0001 C CNN
 F 3 "~" H 2550 5200 50  0001 C CNN
 	1    2550 5200
@@
 	5400 3250 5800 3250
 $Comp
-L power:+BATT #PWR04
-U 1 1 5B621946
-P 5400 3250
-F 0 "#PWR04" H 5400 3100 50  0001 C CNN
-F 1 "+BATT" H 5415 3423 50  0000 C CNN
-F 2 "" H 5400 3250 50  0001 C CNN
-F 3 "" H 5400 3250 50  0001 C CNN
-	1    5400 3250
-	1    0    0    -1
-$EndComp
-$Comp
 L power:+3.3V #PWR03
 U 1 1 5B6223CF
@@
 Connection ~ 2450 3250
 $Comp
-L power:+BATT #PWR07
-U 1 1 5B63312A
-P 2250 900
-F 0 "#PWR07" H 2250 750 50  0001 C CNN
-F 1 "+BATT" H 2265 1073 50  0000 C CNN
-F 2 "" H 2250 900 50  0001 C CNN
-F 3 "" H 2250 900 50  0001 C CNN
-	1    2250 900
-	1    0    0    -1
-$EndComp
-Wire Wire Line
-	2250 900  2250 1250
-$Comp
 L Device:CP C1
 U 1 1 5B61C70B
@@
 	10100 2500 8650 2500
 Connection ~ 8650 2500
+$Comp
+L power:+BATT #PWR08
+U 1 1 5B6A12DC
+P 4500 5300
+F 0 "#PWR08" H 4500 5150 50  0001 C CNN
+F 1 "+BATT" H 4515 5473 50  0000 C CNN
+F 2 "" H 4500 5300 50  0001 C CNN
+F 3 "" H 4500 5300 50  0001 C CNN
+	1    4500 5300
+	1    0    0    -1
+$EndComp
+Wire Wire Line
+	4500 5300 4500 5550
+Wire Wire Line
+	4500 5550 5050 5550
+NoConn ~ 2450 1250
+NoConn ~ 2850 2050
+NoConn ~ 2850 1750
+NoConn ~ 2850 1650
+NoConn ~ 2850 2450
+NoConn ~ 2850 2550
+NoConn ~ 2850 2650
+NoConn ~ 2850 2750
+NoConn ~ 2850 2850
+NoConn ~ 2850 2950
+NoConn ~ 1850 2950
+NoConn ~ 1850 2850
+NoConn ~ 1850 2750
+NoConn ~ 1850 2650
+NoConn ~ 1850 2550
+NoConn ~ 1850 2450
+NoConn ~ 1850 2350
+NoConn ~ 1850 2250
+NoConn ~ 1850 1750
+NoConn ~ 1850 1650
+Wire Wire Line
+	5650 5550 6000 5550
+Wire Wire Line
+	6150 5550 6150 5350
+$Comp
+L Device:R R2
+U 1 1 5B6A1D1C
+P 5350 6100
+F 0 "R2" V 5143 6100 50  0000 C CNN
+F 1 "1.2K" V 5234 6100 50  0000 C CNN
+F 2 "Resistor_SMD:R_0805_2012Metric_Pad1.15x1.40mm_HandSolder" V 5280 6100 50  0001 C CNN
+F 3 "~" H 5350 6100 50  0001 C CNN
+	1    5350 6100
+	-1   0    0    1
+$EndComp
+$Comp
+L power:GND #PWR09
+U 1 1 5B6A1D23
+P 5350 6250
+F 0 "#PWR09" H 5350 6000 50  0001 C CNN
+F 1 "GND" H 5355 6077 50  0000 C CNN
+F 2 "" H 5350 6250 50  0001 C CNN
+F 3 "" H 5350 6250 50  0001 C CNN
+	1    5350 6250
+	1    0    0    -1
+$EndComp
+Wire Wire Line
+	5350 5850 5350 5900
+$Comp
+L Device:R R3
+U 1 1 5B6A2882
+P 5850 5900
+F 0 "R3" V 5643 5900 50  0000 C CNN
+F 1 "240" V 5734 5900 50  0000 C CNN
+F 2 "Resistor_SMD:R_0805_2012Metric_Pad1.15x1.40mm_HandSolder" V 5780 5900 50  0001 C CNN
+F 3 "~" H 5850 5900 50  0001 C CNN
+	1    5850 5900
+	0    -1   -1   0
+$EndComp
+Wire Wire Line
+	5350 5900 5700 5900
+Connection ~ 5350 5900
+Wire Wire Line
+	5350 5900 5350 5950
+Wire Wire Line
+	6000 5900 6000 5550
+Connection ~ 6000 5550
+Wire Wire Line
+	6000 5550 6150 5550
+$Comp
+L power:VCC #PWR0101
+U 1 1 5B6A443D
+P 2250 950
+F 0 "#PWR0101" H 2250 800 50  0001 C CNN
+F 1 "VCC" H 2267 1123 50  0000 C CNN
+F 2 "" H 2250 950 50  0001 C CNN
+F 3 "" H 2250 950 50  0001 C CNN
+	1    2250 950
+	1    0    0    -1
+$EndComp
+Wire Wire Line
+	2250 950  2250 1250
+$Comp
+L power:VCC #PWR0103
+U 1 1 5B6A4B6A
+P 6150 5350
+F 0 "#PWR0103" H 6150 5200 50  0001 C CNN
+F 1 "VCC" H 6167 5523 50  0000 C CNN
+F 2 "" H 6150 5350 50  0001 C CNN
+F 3 "" H 6150 5350 50  0001 C CNN
+	1    6150 5350
+	1    0    0    -1
+$EndComp
+$Comp
+L power:VCC #PWR0106
+U 1 1 5B6A4F66
+P 5400 3000
+F 0 "#PWR0106" H 5400 2850 50  0001 C CNN
+F 1 "VCC" H 5417 3173 50  0000 C CNN
+F 2 "" H 5400 3000 50  0001 C CNN
+F 3 "" H 5400 3000 50  0001 C CNN
+	1    5400 3000
+	1    0    0    -1
+$EndComp
+Wire Wire Line
+	5400 3250 5400 3000
+$Comp
+L Regulator_Linear:LM317_3PinPackage U2
+U 1 1 5B8AB368
+P 5350 5550
+F 0 "U2" H 5350 5792 50  0000 C CNN
+F 1 "LM317_3PinPackage" H 5350 5701 50  0000 C CNN
+F 2 "Package_TO_SOT_THT:TO-220-3_Vertical" H 5350 5800 50  0001 C CIN
+F 3 "http://www.ti.com/lit/ds/symlink/lm317.pdf" H 5350 5550 50  0001 C CNN
+	1    5350 5550
+	1    0    0    -1
+$EndComp
 $EndSCHEMATC
